File: Pixel_click/pixel_click.kicad_sch (KiCad schematic)
At the start: 131 parts, among them J1 USB_C_Receptacle, J2 Conn_01x03_Pin, SW1 boot, SW2 btn1, SW3 btn1, SW4 SW_MEC_5G, SW5 btn1, U1 ESP32-S3, U2 USBLC6-2P6, U3 W25Q128JVS, U4 TLV76733DRVx, U5 SN74LV1T34DBV, Y1 Crystal_GND24_Small

Commit message: Add files via upload
Parts:
- removed SW1: boot, symbol Switch:SW_MEC_5G
- removed SW2, SW3, SW5: btn1, symbol Switch:SW_MEC_5G
- removed SW4: SW_MEC_5G, symbol Switch:SW_MEC_5G
- added SW1: btn4, Button_Switch_THT:SW_Tactile_SPST_Angled_PTS645Vx39-2LFS, symbol Switch:SW_Push
- added SW2: btn3, Button_Switch_THT:SW_Tactile_SPST_Angled_PTS645Vx39-2LFS, symbol Switch:SW_Push
- added SW3: btn2, Button_Switch_THT:SW_Tactile_SPST_Angled_PTS645Vx39-2LFS, symbol Switch:SW_Push
- added SW4: btn5, Button_Switch_THT:SW_Tactile_SPST_Angled_PTS645Vx39-2LFS, symbol Switch:SW_Push
- added SW5: btn1, Button_Switch_THT:SW_Tactile_SPST_Angled_PTS645Vx39-2LFS, symbol Switch:SW_Push
- added TP2, TP3, TP4, TP5, TP6, TP7: TestPoint, symbol Connector:TestPoint
- ANT1: footprint 2450AT18D0100E:DFN320X160X120-4RN -> ANT1:DFN320X160X120-4RN
- C1, C10, C11, C12, C13, C14, C15, C16, C17, C18, C19, C2, C20, C21, C22, C23, C24, C25, C26, C27, C28, C29, C3, C30, C31, C32, C33, C34, C35, C36, C37, C38, C39, C4, C40, C41, C42, C43, C44, C45, C46, C47, C48, C49, C5, C50, C51, C52, C53, C54, C55, C56, C57, C58, C6, C7, C8, C9: footprint (none) -> Capacitor_SMD:C_0201_0603Metric
- D37: footprint (none) -> LED_SMD:LED_0201_0603Metric
- D38: footprint (none) -> LED_SMD:LED_0402_1005Metric
- J1: footprint (none) -> Connector_USB:USB_C_Receptacle_Amphenol_12401548E4-2A
- J2: footprint (none) -> Connector_PinHeader_1.27mm:PinHeader_1x03_P1.27mm_Horizontal
- L1: footprint (none) -> Inductor_SMD:L_0201_0603Metric
- L2: value L -> 2nH; footprint (none) -> Inductor_SMD:L_0201_0603Metric
- NT1: footprint (none) -> NetTie:NetTie-2_SMD_Pad0.5mm
- R1, R10, R11, R12, R13, R14, R15, R16, R17, R2, R3, R4, R5, R6, R7, R8, R9: footprint (none) -> Resistor_SMD:R_0201_0603Metric
- TP1: footprint (none) -> TestPoint:TestPoint_Bridge_Pitch2.0mm_Drill0.7mm
- Y1: footprint (none) -> Crystal_Oscillator:XTAL_ECS-400-10-37B2-CKY-TR
Connections:
- net +3.3V: no longer C55.2, L2.2
- net BOOT: now also SW1.1, TP7.1
- net BTN_1: now also SW5.1
- net BTN_2: now also SW3.1
- net BTN_3: now also SW2.1
- net ESP_D+: now also TP6.1
- net ESP_D-: now also TP5.1
- net GND: now also SW1.2, SW2.2, SW3.2, SW4.2, SW5.2
- net RESET: now also SW4.1, TP4.1
- net VDD3P3: now also C55.2, L2.2
- new net RX: TP3.1
- new net TX: TP2.1
Other:
- moved on the sheet: R9
