File: Pixel_click/pixel_click.kicad_pcb (KiCad board)
At the start: 4 copper layers, 131 parts, among them J1 USB_C_Receptacle, J2 Conn_01x03_Pin, SW1 btn4, SW2 btn3, SW3 btn2, SW4 btn5, SW5 btn1, U1 ESP32-S3, U2 USBLC6-2P6, U3 W25Q128JVS, U4 TLV76733DRVx, U5 SN74LV1T34DBV, Y1 Crystal_GND24_Small

Commit message: Add files via upload
Parts:
- D1, D10, D11, D12, D13, D14, D15, D16, D17, D18, D19, D2, D20, D21, D22, D23, D24, D25, D26, D27, D28, D29, D3, D30, D31, D32, D33, D34, D35, D36, D4, D5, D6, D7, D8, D9: footprint LED_SMD:LED_SK6805_PLCC4_2.4x2.7mm_P1.3mm -> LED_SMD:LED_SK6812_PLCC4_5.0x5.0mm_P3.2mm
- D38: footprint LED_SMD:LED_0402_1005Metric -> LED_SMD:LED_0201_0603Metric
- J2: footprint Connector_PinHeader_1.27mm:PinHeader_1x03_P1.27mm_Horizontal -> Connector_PinHeader_1.27mm:PinHeader_1x03_P1.27mm_Vertical
- SW1, SW2, SW3, SW4, SW5: footprint Button_Switch_THT:SW_Tactile_SPST_Angled_PTS645Vx39-2LFS -> Button_Switch_THT:SW_PUSH_6mm_H4.3mm
- moved R12 84.6 mm to (176.2, 114.6), turned to -90 degrees
- moved C35 83.3 mm to (170.3, 89.5)
- moved ANT1 82.4 mm to (155.6, 72.8)
- moved L1 82.4 mm to (145.6, 71.4)
- moved C38 82.4 mm to (150.4, 72.3)
- moved C39 82.4 mm to (149.2, 72.3)
- moved C40 82.4 mm to (148.0, 72.3)
- moved C41 82.4 mm to (146.6, 72.4)
- moved R13 82.4 mm to (152.0, 72.1)
- moved C33 82.0 mm to (170.3, 103.2)
- moved SW5 81.9 mm to (175.7, 121.3)
- moved D36 81.8 mm to (164.5, 80.9), turned to 0 degrees
- moved C44 81.5 mm to (171.8, 88.0)
- moved J2 81.5 mm to (174.7, 86.3)
- moved D5 81.0 mm to (164.5, 87.6), turned to 180 degrees
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Connections:
- U1 pad 24: /BTN_1 -> unconnected-(U1-GPIO21-Pad24)
- U1 pad 27: unconnected-(U1-GPIO21-Pad27) -> /BTN_1
- U1 pad 28: unconnected-(U1-SPICS1-Pad28) -> /BTN_3
- U1 pad 9: /BTN_3 -> unconnected-(U1-SPICS1-Pad9)
Routing:
- net GND: track 250.1 -> 507.3 mm, vias 51 -> 36
- net +3.3V: track 163.6 -> 318.1 mm, vias 4 -> 5
- net /LED_DATA_5V: track 0.00 -> 150.1 mm, vias 0 -> 1
- net /LED_DATA_3V3: track 2.02 -> 147.0 mm, vias 0 -> 1
- net /BTN_3: track 6.20 -> 93.1 mm, vias 0 -> 1
- net /BTN_1: track 5.59 -> 48.9 mm
- net /BOOT: track 24.1 -> 65.3 mm, vias 2 -> 0
- net +5V: track 543.5 -> 581.1 mm, vias 10 -> 12
- net /VBUS: track 5.37 -> 19.9 mm
- net Net-(U1-SPIHD): track 23.8 -> 11.5 mm
- net /LNA_IN: track 19.5 -> 29.2 mm
- net Net-(U1-SPICLK): track 22.0 -> 12.5 mm
- net Net-(U1-SPIQ): track 22.2 -> 12.7 mm
- net Net-(U1-SPIWP): track 23.1 -> 13.7 mm
- net Net-(U1-SPID): track 21.8 -> 12.9 mm
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Other:
- board outline added: 82.4 x 59.6 mm
