File: BBBC/BBBC.kicad_pcb (KiCad board)
At the start: 2 copper layers, 76.8 x 32.8 mm, 24 parts, among them J1 Screw_Terminal_01x02, J2 Screw_Terminal_01x02, Q1 IRF540N, U1 TL494, U2 ADA4610-1xRJ

Commit message: Add files via upload
Parts:
- added REF**: Symbol_HighVoltage_NoTriangle_6x15mm_Copper, Symbol:Symbol_HighVoltage_NoTriangle_6x15mm_Copper, F.Cu at (73.5, 80.5)
Changed lines of the file:
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@@
 		(tags "Resistor Axial_DIN0204 series Axial Horizontal pin pitch 5.08mm 0.167W length 3.6mm diameter 1.6mm")
 		(property "Reference" "R6"
-			(at 2.54 -1.92 360)
+			(at 2.54 -1.92 0)
 			(layer "F.SilkS")
 			(hide yes)
@@
 		)
 		(property "Value" "560R"
-			(at 2.54 1.92 360)
+			(at 2.54 1.92 0)
 			(layer "F.Fab")
 			(hide yes)
@@
 		)
 		(fp_text user "${REFERENCE}"
-			(at 2.54 0 360)
+			(at 2.54 0 0)
 			(layer "F.Fab")
 			(effects
@@
 		(tags "C Rect series Radial pin pitch 2.50mm  length 4.6mm width 2mm Capacitor")
 		(property "Reference" "C3"
-			(at 1.25 -2.25 360)
+			(at 1.25 -2.25 0)
 			(layer "F.SilkS")
 			(hide yes)
@@
 		)
 		(property "Value" "2.2nF"
-			(at 1.25 2.25 360)
+			(at 1.25 2.25 0)
 			(layer "F.Fab")
 			(hide yes)
@@
 		)
 		(fp_text user "${REFERENCE}"
-			(at 1.25 0 360)
+			(at 1.25 0 0)
 			(layer "F.Fab")
 			(effects
@@
 		)
 	)
+	(footprint "Symbol:Symbol_HighVoltage_NoTriangle_6x15mm_Copper"
+		(layer "F.Cu")
+		(at 73.55 80.45)
+		(descr "High voltage symbol, no triangle, 6x15mm, copper layer")
+		(tags "warning graphic")
+		(property "Reference" "REF**"
+			(at 0 -8.5 0)
+			(layer "F.SilkS")
+			(hide yes)
+			(effects
+				(font
+					(size 1 1)
+					(thickness 0.15)
+				)
+			)
+		)
+		(property "Value" "Symbol_HighVoltage_NoTriangle_6x15mm_Copper"
+			(at -1.27 8.5 0)
+			(layer "F.Fab")
+			(hide yes)
+			(effects
+				(font
+					(size 1 1)
+					(thickness 0.15)
+				)
+			)
+		)
+		(property "Footprint" "Symbol:Symbol_HighVoltage_NoTriangle_6x15mm_Copper"
+			(at 0 0 0)
+			(unlocked yes)
+			(layer "F.Fab")
+			(hide yes)
+			(effects
+				(font
+					(size 1.27 1.27)
+					(thickness 0.15)
+				)
+			)
+		)
+		(property "Datasheet" ""
+			(at 0 0 0)
+			(unlocked yes)
+			(layer "F.Fab")
+			(hide yes)
+			(effects
+				(font
+					(size 1.27 1.27)
+					(thickness 0.15)
+				)
+			)
+		)
+		(property "Description" ""
+			(at 0 0 0)
+			(unlocked yes)
+			(layer "F.Fab")
+			(hide yes)
+			(effects
+				(font
+					(size 1.27 1.27)
+					(thickness 0.15)
+				)
+			)
+		)
+		(attr exclude_from_pos_files exclude_from_bom allow_missing_courtyard)
+		(fp_poly
+			(pts
+				(xy -0.77 4.54) (xy 1.07 4.98) (xy -0.333376 7.501)
+			)
+			(stroke
+				(width 0.2)
+				(type solid)
+			)
+			(fill solid)
+			(layer "F.Cu")
+		)
+		(fp_poly
+			(pts
+				(xy 0.619125 -0.547625) (xy 0.13 -0.28) (xy 0.55 0.02)
+			)
+			(stroke
+				(width 0.2)
+				(type solid)
+			)
+			(fill solid)
+			(layer "F.Cu")
+		)
+		(fp_poly
+			(pts
+				(xy -0.88 -1.14) (xy -1.143 -0.5) (xy -0.52 -0.81) (xy -0.89 -1.14)
+			)
+			(stroke
+				(width 0.2)
+				(type solid)
+			)
+			(fill solid)
+			(layer "F.Cu")
+		)
+		(fp_poly
+			(pts
+				(xy -1.143 -0.5) (xy 2.666999 -2.547875) (xy 0.523874 5.262625) (xy 1.61925 4.595875) (xy -0.333376 7.501)
+				(xy -1.04775 4.072001) (xy -0.285751 5.11975) (xy 0.619125 -0.547625) (xy -3.048001 1.405001) (xy -0.666751 -7.024625)
+				(xy 1.666874 -7.024625)
+			)
+			(stroke
+				(width 0.2)
+				(type solid)
+			)
+			(fill solid)
+			(layer "F.Cu")
+		)
+	)
 	(footprint "Resistor_THT:R_Axial_DIN0204_L3.6mm_D1.6mm_P5.08mm_Horizontal"
 		(layer "F.Cu")
@@
 		(tags "SOT TO_SOT_SMD")
 		(property "Reference" "U2"
-			(at 0 -2.4 360)
+			(at 0 -2.4 0)
 			(layer "F.SilkS")
 			(hide yes)
@@
 		)
 		(property "Value" "ADA4610-1xRJ"
-			(at 0 2.4 360)
+			(at 0 2.4 0)
 			(layer "F.Fab")
 			(hide yes)
@@
 		)
 		(fp_text user "${REFERENCE}"
-			(at 0 0 360)
+			(at 0 0 0)
 			(layer "F.Fab")
 			(effects
@@
 		(tags "Resistor Axial_DIN0204 series Axial Horizontal pin pitch 5.08mm 0.167W length 3.6mm diameter 1.6mm")
 		(property "Reference" "R11"
-			(at 2.54 -1.92 360)
+			(at 2.54 -1.92 0)
 			(layer "F.SilkS")
 			(hide yes)
@@
 		)
 		(property "Value" "10K"
-			(at 2.54 1.92 360)
+			(at 2.54 1.92 0)
 			(layer "F.Fab")
 			(hide yes)
@@
 		)
 		(fp_text user "${REFERENCE}"
-			(at 2.54 0 360)
+			(at 2.54 0 0)
 			(layer "F.Fab")
 			(effects
@@
 		(tags "Ferrite vertical LairdTech 28C0236-0JW-10")
 		(property "Reference" "L1"
-			(at 2.54 -4.064 360)
+			(at 2.54 -4.064 0)
 			(layer "F.SilkS")
 			(hide yes)
@@
 		)
 		(property "Value" "220uH"
-			(at 2.54 4.953 360)
+			(at 2.54 4.953 0)
 			(layer "F.Fab")
 			(hide yes)
@@
 		)
 		(fp_text user "${REFERENCE}"
-			(at 2.54 0 360)
+			(at 2.54 0 0)
 			(layer "F.Fab")
 			(effects
